File: Hardware/Schematic/Schematic.kicad_sch (KiCad schematic)
At the start: 3 parts, among them U1 OLED Display, U2 Analog Microphone

Commit message: aaa
Parts:
- added SW1, SW2: SW_Push, symbol Switch:SW_Push
Connections:
- net GND: now also SW1.2, SW2.2
- net at A1.24 (GPIO18): now also SW1.1
- net at A1.34 (GPIO28_ADC2): now also SW2.1
- no-connect marks 0 -> 27
